File: Hackpad.kicad_sch (KiCad schematic)
At the start: 0 parts

Commit message: Created schematic and PCB
PCB is still not routed.
Parts:
- added D1, D2, D3, D4: SK6812MINI, LED_SMD:LED_SK6812MINI_PLCC4_3.5x3.5mm_P1.75mm, symbol LED:SK6812MINI
- added SW1, SW2, SW3, SW4: SW_Push, Button_Switch_Keyboard:SW_Cherry_MX_1.00u_PCB, symbol Switch:SW_Push
- added SW5: RotaryEncoder, Rotary_Encoder:RotaryEncoder_Alps_EC11E_Vertical_H20mm, symbol Device:RotaryEncoder
- added U1: XIAO-RP2040-DIP, Seeed Studio XIAO Series Library:XIAO-RP2040-DIP, symbol Seeed_Studio_XIAO_Series:XIAO-RP2040-DIP
- added U2: SSD1306, KiCad-SSD1306-0.91-OLED-4pin-128x32.pretty-master:SSD1306-0.91-OLED-4pin-128x32, symbol OLED0.91:OLED_0.91
Connections:
- new net: D1.1 (DOUT), D2.3 (DIN)
- new net: D1.3 (DIN), U1.1 (GPIO26/ADC0/A0)
- new net: SW5.A, U1.2 (GPIO27/ADC1/A1)
- new net: SW5.B, U1.3 (GPIO28/ADC2/A2)
- new net: SW1.2, U1.8 (GPIO1/RX)
- new net: SW3.2, U1.10 (GPIO4/MISO)
- new net: SW4.2, U1.11 (GPIO3/MOSI)
- new net: U1.5 (GPIO6/SDA), U2.3 (SDA)
- new net: U1.6 (GPIO7/SCL), U2.4 (SCL)
- new net: SW2.2, U1.9 (GPIO2/SCK)
- new net: D3.1 (DOUT), D4.3 (DIN)
- new net: D2.1 (DOUT), D3.3 (DIN)
- new net +5V: D1.4 (VDD), D2.4 (VDD), D3.4 (VDD), D4.4 (VDD), U1.14 (VBUS), U2.1 (VCC)
- new net GND: D1.2 (VSS), D2.2 (VSS), D3.2 (VSS), D4.2 (VSS), SW1.1, SW2.1, SW3.1, SW4.1, SW5.C, U1.13 (GND), U2.2 (GND)
